File: hardware/module.kicad_pcb (KiCad board)
At the start: 2 copper layers, 59.2 x 33 mm, 41 parts, among them J2 PROG, J3 PRB1, J4 PRB2, P1 USB_C_Plug_USB2.0, SW1 RESET, U1 STM32L010C6Tx, U2 CP2102N-Axx-xQFN20, U3 USBLC6-2P6, U4 TMUX6236, U5 EZO-EC™, U6 SI8600AB-B-IS, U7 TPS631000, U8 PCIEx4

Commit message: Update PCB module design
Co-authored-by: Kshitij Dadhekar <kshitij.dadhekar@clearwings.nl>
Parts:
- removed J2: PROG, Connector:Tag-Connect_TC2030-IDC-NL_2x03_P1.27mm_Vertical
- removed J4: PRB2, Connector_Coaxial:SMA_Molex_73251-1153_EdgeMount_Horizontal
- added C12: 100n, Capacitor_SMD:C_0603_1608Metric, F.Cu at (141.4, 54.9)
- added C13: 100n, Capacitor_SMD:C_0603_1608Metric, F.Cu at (143.2, 65.9)
- added C14: 100n, Capacitor_SMD:C_0603_1608Metric, F.Cu at (152.4, 53.0)
- added C15: 100n, Capacitor_SMD:C_0603_1608Metric, F.Cu at (155.6, 49.7)
- added C16: 4u7, Capacitor_SMD:C_0603_1608Metric, F.Cu at (155.6, 53.0)
- added C17: 4u7, Capacitor_SMD:C_0603_1608Metric, F.Cu at (155.6, 51.3)
- added C18: 47u, Capacitor_SMD:C_0805_2012Metric, F.Cu at (178.9, 50.2)
- added C19: 4u7, Capacitor_SMD:C_0603_1608Metric, F.Cu at (177.0, 50.5)
- added C20: 47u, Capacitor_SMD:C_0805_2012Metric, F.Cu at (170.1, 54.6)
- added C21: 4u7, Capacitor_SMD:C_0603_1608Metric, F.Cu at (170.1, 56.3)
- added C22: 10u, Capacitor_SMD:C_0603_1608Metric, F.Cu at (156.7, 68.2)
- added C23: 10u, Capacitor_SMD:C_0603_1608Metric, F.Cu at (159.6, 74.6)
- added D1: MBR0520LT1G, Diode_SMD:D_SOD-123, F.Cu at (155.9, 73.9)
- added D2: MBR0520LT1G, Diode_SMD:D_SOD-123, F.Cu at (169.6, 51.3)
- added D3: MBR0520LT1G, Diode_SMD:D_SOD-123, F.Cu at (159.7, 71.8)
- added D4: MBR0520LT1G, Diode_SMD:D_SOD-123, F.Cu at (170.6, 58.2)
- added FID1: Fiducial, Fiducial:Fiducial_0.5mm_Mask1mm, F.Cu at (146.8, 80.0)
- added FID2: Fiducial, Fiducial:Fiducial_0.5mm_Mask1mm, F.Cu at (192.8, 65.3)
- added J1: Conn_ARM_JTAG_SWD_10, Connector:Tag-Connect_TC2050-IDC-NL_2x05_P1.27mm_Vertical, F.Cu at (188.3, 69.8)
- added J6: CON-SMA-EDGE-S, CON-SMA-EDGE-S:RFSOLUTIONS_CON-SMA-EDGE-S, F.Cu at (137.3, 61.2)
- added J7: CON-SMA-EDGE-S, CON-SMA-EDGE-S:RFSOLUTIONS_CON-SMA-EDGE-S, F.Cu at (137.3, 52.0)
- added R15: 2K2, Resistor_SMD:R_0603_1608Metric, F.Cu at (170.5, 70.0)
- added R16: 2K2, Resistor_SMD:R_0603_1608Metric, F.Cu at (173.6, 74.8)
- added R17: 0R, Resistor_SMD:R_0603_1608Metric, F.Cu at (172.0, 74.8)
- added R18: 0R, Resistor_SMD:R_0603_1608Metric, F.Cu at (170.4, 74.8)
- added R19: 0R, Resistor_SMD:R_0603_1608Metric, F.Cu at (179.3, 74.8)
- added R20: 0R, Resistor_SMD:R_0603_1608Metric, F.Cu at (180.9, 74.8)
- added R21: 0R, Resistor_SMD:R_0603_1608Metric, F.Cu at (182.5, 74.8)
- added R22: 0R, Resistor_SMD:R_0603_1608Metric, F.Cu at (170.0, 61.7)
- added R23: 10k, Resistor_SMD:R_0603_1608Metric, F.Cu at (170.0, 63.2)
- added R24: 5k2, Resistor_SMD:R_0603_1608Metric, F.Cu at (144.8, 77.7)
- added R25: 5k2, Resistor_SMD:R_0603_1608Metric, F.Cu at (144.8, 76.0)
- added TP1: TestPoint, TestPoint:TestPoint_Pad_1.0x1.0mm, B.Cu at (187.2, 53.2)
- added TP10: TestPoint, TestPoint:TestPoint_Pad_1.0x1.0mm, B.Cu at (161.2, 58.7)
- added TP11: TestPoint, TestPoint:TestPoint_Pad_1.0x1.0mm, B.Cu at (166.5, 69.0)
- added TP12: TestPoint, TestPoint:TestPoint_Pad_1.0x1.0mm, B.Cu at (166.2, 54.5)
- added TP13: TestPoint, TestPoint:TestPoint_Pad_1.0x1.0mm, B.Cu at (178.3, 59.6)
- added TP14: TestPoint, TestPoint:TestPoint_Pad_1.0x1.0mm, B.Cu at (180.6, 59.6)
- added TP15: TestPoint, TestPoint:TestPoint_Pad_1.0x1.0mm, B.Cu at (142.2, 67.2)
- added TP16: TestPoint, TestPoint:TestPoint_Pad_1.0x1.0mm, B.Cu at (142.5, 76.3)
- added TP2: TestPoint, TestPoint:TestPoint_Pad_1.0x1.0mm, B.Cu at (178.2, 53.9)
- added TP3: TestPoint, TestPoint:TestPoint_Pad_1.0x1.0mm, B.Cu at (153.4, 75.5)
- added TP4: TestPoint, TestPoint:TestPoint_Pad_1.0x1.0mm, B.Cu at (166.2, 56.6)
- added TP5: TestPoint, TestPoint:TestPoint_Pad_1.0x1.0mm, B.Cu at (147.3, 53.0)
- added TP6: TestPoint, TestPoint:TestPoint_Pad_1.0x1.0mm, B.Cu at (144.6, 50.5)
- added TP7: TestPoint, TestPoint:TestPoint_Pad_1.0x1.0mm, B.Cu at (159.0, 64.7)
- added TP8: TestPoint, TestPoint:TestPoint_Pad_1.0x1.0mm, B.Cu at (161.6, 54.7)
- added TP9: TestPoint, TestPoint:TestPoint_Pad_1.0x1.0mm, B.Cu at (161.5, 51.6)
- C1: value 100n -> 4u7; footprint Capacitor_SMD:C_0805_2012Metric -> Capacitor_SMD:C_0603_1608Metric
- C10, C11, C3, C4, C5, C6, C7, C8, C9: footprint Capacitor_SMD:C_0805_2012Metric -> Capacitor_SMD:C_0603_1608Metric
- C2: value 47u -> 10u; footprint Capacitor_SMD:C_0805_2012Metric -> Capacitor_SMD:C_0603_1608Metric
- J3: value PRB1 -> Screw_Terminal_01x06; footprint Connector_Coaxial:SMA_Molex_73251-1153_EdgeMount_Horizontal -> TerminalBlock_Phoenix:TerminalBlock_Phoenix_MPT-0,5-6-2.54_1x06_P2.54mm_Horizontal
- L1: value 1uH @ 2.1A -> LPWI201208S1R0T
- P1: value USB_C_Plug_USB2.0 -> USB4105-GF-A
- PS1: value IA0505S -> IA0505D; footprint Converter_DCDC:Converter_DCDC_XP_POWER-IAxxxxS_THT -> Converter_DCDC:Converter_DCDC_XP_POWER-IAxxxxD_THT
- R1, R10, R11, R12, R13, R14, R2, R3, R4, R5, R6, R7, R9: footprint Resistor_SMD:R_0805_2012Metric -> Resistor_SMD:R_0603_1608Metric
- R8: value 27 -> 10k; footprint Resistor_SMD:R_0805_2012Metric -> Resistor_SMD:R_0603_1608Metric
- SW1: value RESET -> PTS810SJG250SMTRLFS; footprint Button_Switch_SMD:SW_SPST_CK_RS282G05A3 -> Button_Switch_SMD:SW_SPST_PTS810
- U1: value STM32L010C6Tx -> STM32L010C6T6
- U2: value CP2102N-Axx-xQFN20 -> CP2102N-A02-GQFN20
- U3: footprint Package_TO_SOT_SMD:SOT-666 -> USBLC6-2P6:SOT50P160X60-6N
- U4: value TMUX6236 -> TMUX6236PWR
- U6: value SI8600AB-B-IS -> ISO1644DWR; footprint Package_SO:SOIC-8_3.9x4.9mm_P1.27mm -> Package_SO:SOIC-16W_7.5x10.3mm_P1.27mm
- U7: value TPS631000 -> TPS631000DRLR
- moved R13 25.5 mm to (146.6, 71.0), turned to 0 degrees
- moved C4 24.1 mm to (155.1, 68.2), turned to -90 degrees
- moved R3 22.2 mm to (172.2, 50.5), turned to 90 degrees
- moved R12 22.2 mm to (151.0, 70.9), turned to 180 degrees
- moved C5 20.3 mm to (144.8, 65.9)
- moved R5 19.5 mm to (173.8, 50.5), turned to -90 degrees
- moved U6 18.7 mm to (151.6, 59.5)
- moved R14 18.4 mm to (175.2, 74.8), turned to 90 degrees
- moved JP1 17.7 mm to (177.2, 74.8), turned to -90 degrees
- moved R4 17.2 mm to (175.4, 50.5)
- moved U4 15.3 mm to (142.7, 59.8), turned to -90 degrees
- moved U2 14.8 mm to (174.3, 55.6), turned to 180 degrees
- moved C9 14.5 mm to (170.0, 66.8), turned to 180 degrees
- moved R11 13.7 mm to (183.8, 60.8), turned to 90 degrees
- moved R10 13.6 mm to (185.5, 60.8), turned to 90 degrees
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Connections:
- net Net-(U2-D+) renamed /CP_P
- net Net-(U2-D-) renamed /CP_N
- net Net-(U2-VDD) renamed CP2102_3V3
- net Net-(U2-VREGIN) renamed USB_VBUS
- C10 pad 1: VSensor -> 3V3
- C11 pad 1: VSensor -> 3V3
- C3 pad 1: Net-(U7-Vin) -> 3V3
- C4 pad 1: VSensor -> 3V3
- C7 pad 1: VSensor -> 3V3
- C8 pad 1: VSensor -> 3V3
- C9 pad 1: VSensor -> 3V3
- J3 pad 1: Net-(J3-In) -> +5V_ISO
- J3 pad 2: Net-(J3-Ext) -> /DQ_TEMP_B_ISO
- JP1 pad 2: VSensor -> 3V3
- P1 pad A6: Net-(P1-D+) -> /USB_P
- P1 pad A7: Net-(P1-D-) -> /USB_N
- P1 pad B6: (no net) -> /USB_P
- P1 pad B7: (no net) -> /USB_N
- PS1 pad 1: +5V -> GND
- PS1 pad 2: GND -> unconnected-(PS1-NC-Pad2)
- PS1 pad 5: GND_ISO -> +5V_ISO
- PS1 pad 6: +5V_ISO -> GND_ISO
- R10 pad 1: VSensor -> /LPUART1_TX
- R10 pad 2: /LPUART1_TX -> 3V3
- R11 pad 1: VSensor -> /LPUART1_RX
- R11 pad 2: /LPUART1_RX -> 3V3
- R12 pad 2: Net-(U5-RX/SCL) -> Net-(U5-TX/SDA)
- R13 pad 2: Net-(U5-TX/SDA) -> Net-(U5-RX/SCL)
- R8 pad 1: Net-(U7-Vin) -> Net-(U4-EN)
- R8 pad 2: VSensor -> +5V_ISO
- U1 pad 15: unconnected-(U1-PA5-Pad15) -> /DQ_TEMP_A
- U1 pad 16: unconnected-(U1-PA6-Pad16) -> /PRB_SEL_MCU
- U1 pad 17: unconnected-(U1-PA7-Pad17) -> /DQ_TEMP_B
- U1 pad 24: VSensor -> 3V3
- U1 pad 25: unconnected-(U1-PB12-Pad25) -> Net-(U1-PB12)
- U1 pad 36: VSensor -> 3V3
- U1 pad 41: unconnected-(U1-PB5-Pad41) -> Net-(U1-PB5)
- U1 pad 42: /I2C_SCL -> Net-(U1-PB6)
- U1 pad 43: /I2C_SDA -> Net-(U1-PB7)
- U1 pad 45: unconnected-(U1-PB8-Pad45) -> Net-(U1-PB8)
- U1 pad 46: unconnected-(U1-PB9-Pad46) -> Net-(U1-PB9)
- U1 pad 48: VSensor -> 3V3
- U1 pad 9: VSensor -> 3V3
- U3 pad 4: Net-(P1-D+) -> /USB_P
- U3 pad 6: Net-(P1-D-) -> /USB_N
- U4 pad 1: /PRB_SEL_A -> /PRB_SEL
- U4 pad 10: Net-(J3-Ext) -> Net-(U4-S2A)
- U4 pad 14: /PRB_EN -> Net-(U4-EN)
- U4 pad 2: Net-(J3-In) -> Net-(U4-S1A)
- U4 pad 9: /PRB_SEL_B -> /PRB_SEL
- U6 pad 1: VSensor -> 3V3
- U6 pad 2: /LPUART1_TX -> GND
- U6 pad 3: /LPUART1_RX -> /DQ_TEMP_A
- U6 pad 4: GND -> /PRB_SEL_MCU
- U6 pad 5: +5V_ISO -> /LPUART1_TX
- U6 pad 6: Net-(U5-TX/SDA) -> /DQ_TEMP_B
- U6 pad 7: Net-(U5-RX/SCL) -> /LPUART1_RX
- U6 pad 8: GND_ISO -> GND
- U7 pad 4: Net-(U7-Vin) -> 3V3
Routing:
- net GND: track 54.7 -> 9.76 mm, vias 21 -> 11
- net 3V3: track 0.00 -> 44.8 mm, vias 0 -> 11
- net USB_VBUS: track 18.4 -> 50.1 mm, vias 0 -> 5
- net /DQ_TEMP_A: track 0.00 -> 30.1 mm, vias 0 -> 2
- net /DQ_TEMP_B: track 0.00 -> 28.6 mm, vias 0 -> 2
- net /DQ_TEMP_A_ISO: track 0.00 -> 28.5 mm, vias 0 -> 1
- net GND_ISO: track 4.25 -> 32.3 mm
- net Net-(D3-K): track 0.00 -> 26.4 mm, vias 0 -> 1
- net /PRB_SEL_MCU: track 0.00 -> 25.9 mm, vias 0 -> 2
- net /DQ_TEMP_B_ISO: track 0.00 -> 25.4 mm, vias 0 -> 2
- net /BOOST_EN: track 2.94 -> 24.8 mm, vias 0 -> 2
- net Net-(U4-D2): track 0.00 -> 20.7 mm, vias 0 -> 1
- net Net-(U4-S2B): track 0.00 -> 19.4 mm, vias 0 -> 1
- net -5V_ISO: track 10.7 -> 28.0 mm, vias 0 -> 3
- net /PRB_SEL: track 0.00 -> 16.6 mm
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- added copper zone on B.Cu, net 3V3
- removed copper zone on F.Cu, net +5V
- removed copper zone on F.Cu, net Net-(U7-LX1)
- removed copper zone on F.Cu, net Net-(U7-LX2)
- removed copper zone on F.Cu, net Net-(U7-Vin)
- removed copper zone on F.Cu, net VSensor
Other:
- board text added: "+"
- board text added: "-"
- board text added: "0"
- board text added: "0 mm"
- board text added: "0,025 mm"
- board text added: "0,029"
- board text added: "0,035"
- board text added: "0,035 mm"
- board text added: "0,1500 mm / 0,1500 mm"
- board text added: "0,3000 mm"
- board text added: "1"
- board text added: "1,55 mm"
- board text added: "1,6700 mm"
- board text added: "2"
- board text added: "3,7"
- board text added: "4,6"
- board text added: "59,2500 mm x 37,5372 mm"
- board text added: "A"
- board text added: "B"
- board text added: "B.Cu"
- board text added: "B.Mask"
- board text added: "B.Paste"
- board text added: "B.Silkscreen"
- board text added: "BOARD CHARACTERISTICS"
- board text added: "Board Thickness:"
- board text added: "Board overall dimensions:"
- board text added: "Bottom Silk Screen"
- board text added: "Bottom Solder Mask"
- board text added: "Bottom Solder Paste"
- board text added: "Castellated pads:"
- board text added: "Color"
- board text added: "Copper Finish:"
- board text added: "Copper Layer Count:"
- board text added: "Dielectric"
- board text added: "Direct Printing"
- board text added: "ENIG"
- board text added: "Edge card connectors:"
- board text added: "Epsilon R"
- board text added: "F.Cu"
- board text added: "F.Mask"
- board text added: "F.Paste"
- board text added: "F.Silkscreen"
- board text added: "FR4"
- board text added: "FR4 natural"
- board text added: "Green"
- board text added: "Impedance Control:"
- board text added: "Layer Name"
- board text added: "Liquid Ink"
- board text added: "Loss Tangent"
- board text added: "Material"
- board text added: "Min hole diameter:"
- board text added: "Min track/spacing:"
- board text added: "No"
- board text added: "PA"
- board text added: "PB"
- board text added: "Plated Board Edge:"
- board text added: "Thickness (mm)"
- board text added: "Top Silk Screen"
- board text added: "Top Solder Mask"
- board text added: "Top Solder Paste"
- board text added: "Type"
- board text added: "White"
- board text added: "Yes"
- board text added: "copper"
- board text added: "core"

Commit message: feat: new shell commands chore: remove saul pins chore: add compile time FW_VERSION docs: add calibration interpolated graphs
Parts:
- removed J1: Conn_ARM_JTAG_SWD_10, Connector:Tag-Connect_TC2050-IDC-NL_2x05_P1.27mm_Vertical
- added J2: GPHD-2X05, Connector_PinHeader_1.27mm:PinHeader_2x05_P1.27mm_Vertical, F.Cu at (190.0, 73.4)
- J3: value Screw_Terminal_01x06 -> 1725698
Routing:
- net /SWDIO: track 16.9 -> 21.0 mm
- net 3V3: track 44.8 -> 43.3 mm, vias 11 -> 10
- net /SWCLK: track 17.6 -> 19.0 mm
- net /NRST: track 21.2 -> 22.3 mm
