File: hardware/sensor_connector.kicad_sch (KiCad schematic)
At the start: 1 part, among them U8 PCIEx4

Commit message: Update PCB module design
Co-authored-by: Kshitij Dadhekar <kshitij.dadhekar@clearwings.nl>
Parts:
- U8: now not fitted
Changed lines of the file:
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@@
 		(in_bom yes)
 		(on_board yes)
-		(dnp no)
+		(dnp yes)
 		(fields_autoplaced yes)
 		(property "Reference" "U8"
